File: Electronics/whale_circuit_1.sch (KiCad schematic (older format))
At the start: 12 parts

Commit message: Finished power diagram.
Parts:
- added D?: STATUS LED, symbol LED
- added SW?: E-Stop, symbol SW_Reed
- TH?: value Thermistor_PTC -> Temp_Sensor
Connections:
- net GND: now also Act.GND1, D?.1 (K)
- net VCC: now also SW?.1
- net at E-STOP.A1: now also Act.8
- net at Sense/Think.0: now also XB?.2 (DOUT)
- net at Sense/Think.1: now also XB?.3 (DIN/~CONFIG)
- net at Sense/Think.SCL: now also Act.SCL
- net at Sense/Think.SDA: now also Act.SDA
- net at Act.13: now also D?.2 (A)
- net at Act.5V: now also SW?.2
Other:
- moved on the sheet: XB?
Changed lines of the file:
@@
 P 1050 12450
 F 0 "TH?" V 890 12450 50  0001 C CNN
-F 1 "Thermistor_PTC" V 1170 12450 50  0000 C CNN
+F 1 "Temp_Sensor" V 1170 12450 50  0000 C CNN
 F 2 "" H 1100 12250 50  0001 L CNN
 F 3 "" H 1050 12450 50  0001 C CNN
@@
 L XBEE XB?
 U 1 1 5A035AF5
-P 2650 8800
-F 0 "XB?" H 2650 9600 60  0000 C CNN
-F 1 "XBEE" H 2650 9700 60  0000 C CNN
-F 2 "" H 2650 8800 60  0000 C CNN
-F 3 "" H 2650 8800 60  0000 C CNN
-	1    2650 8800
-	1    0    0    -1
+P 2750 8250
+F 0 "XB?" H 2750 9050 60  0000 C CNN
+F 1 "XBEE" H 2750 9150 60  0000 C CNN
+F 2 "" H 2750 8250 60  0000 C CNN
+F 3 "" H 2750 8250 60  0000 C CNN
+	1    2750 8250
+	-1   0    0    1
 $EndComp
 $Comp
 L VCC #PWR?
 U 1 1 5A035CB4
-P 1600 8350
-F 0 "#PWR?" H 1600 8200 50  0001 C CNN
-F 1 "VCC" H 1600 8500 50  0000 C CNN
-F 2 "" H 1600 8350 50  0001 C CNN
-F 3 "" H 1600 8350 50  0001 C CNN
-	1    1600 8350
+P 3950 8850
+F 0 "#PWR?" H 3950 8700 50  0001 C CNN
+F 1 "VCC" H 3950 9000 50  0000 C CNN
+F 2 "" H 3950 8850 50  0001 C CNN
+F 3 "" H 3950 8850 50  0001 C CNN
+	1    3950 8850
 	1    0    0    -1
 $EndComp
@@
 L GND #PWR?
 U 1 1 5A0360DA
-P 1600 9250
-F 0 "#PWR?" H 1600 9000 50  0001 C CNN
-F 1 "GND" H 1600 9100 50  0000 C CNN
-F 2 "" H 1600 9250 50  0001 C CNN
-F 3 "" H 1600 9250 50  0001 C CNN
-	1    1600 9250
-	1    0    0    -1
-$EndComp
+P 4000 7800
+F 0 "#PWR?" H 4000 7550 50  0001 C CNN
+F 1 "GND" H 4000 7650 50  0000 C CNN
+F 2 "" H 4000 7800 50  0001 C CNN
+F 3 "" H 4000 7800 50  0001 C CNN
+	1    4000 7800
+	1    0    0    -1
+$EndComp
+Wire Wire Line
+	3950 8850 3800 8700
+Wire Wire Line
+	3800 7800 4000 7800
+Wire Wire Line
+	3800 8600 4400 8600
+Wire Wire Line
+	4400 8600 4400 12950
+Wire Wire Line
+	4600 8500 4600 12850
+Wire Wire Line
+	4600 8500 3800 8500
+Wire Wire Line
+	4400 12950 3550 12950
+Wire Wire Line
+	4600 12850 3550 12850
+Wire Wire Line
+	3550 11150 5700 11150
+Wire Wire Line
+	5700 11150 5700 11000
+Wire Wire Line
+	5700 11000 7450 11000
+Wire Wire Line
+	7450 11000 7450 11150
+Wire Wire Line
+	7450 11250 7550 11250
+Wire Wire Line
+	7550 11250 7550 10950
+Wire Wire Line
+	7550 10950 5600 10950
+Wire Wire Line
+	5600 10950 5600 11250
+Wire Wire Line
+	5600 11250 3550 11250
+Wire Wire Line
+	5950 14250 7650 14250
+Wire Wire Line
+	7650 14250 7650 12050
+Wire Wire Line
+	7650 12050 7450 12050
+$Comp
+L SW_Reed SW?
+U 1 1 5A0E6483
+P 5250 11900
+F 0 "SW?" H 5250 12000 50  0001 C CNN
+F 1 "E-Stop" H 5250 11800 50  0000 C CNN
+F 2 "" H 5250 11900 50  0001 C CNN
+F 3 "" H 5250 11900 50  0001 C CNN
+	1    5250 11900
+	1    0    0    -1
+$EndComp
+Wire Wire Line
+	5550 11950 5450 11900
+$Comp
+L VCC #PWR?
+U 1 1 5A0E656E
+P 4900 11850
+F 0 "#PWR?" H 4900 11700 50  0001 C CNN
+F 1 "VCC" H 4900 12000 50  0000 C CNN
+F 2 "" H 4900 11850 50  0001 C CNN
+F 3 "" H 4900 11850 50  0001 C CNN
+	1    4900 11850
+	1    0    0    -1
+$EndComp
+Wire Wire Line
+	4900 11850 4900 11900
+Wire Wire Line
+	4900 11900 5050 11900
+Wire Wire Line
+	5400 12100 5550 12050
+$Comp
+L GND #PWR?
+U 1 1 5A0E68D1
+P 5400 12100
+F 0 "#PWR?" H 5400 11850 50  0001 C CNN
+F 1 "GND" H 5400 11950 50  0000 C CNN
+F 2 "" H 5400 12100 50  0001 C CNN
+F 3 "" H 5400 12100 50  0001 C CNN
+	1    5400 12100
+	1    0    0    -1
+$EndComp
+Wire Wire Line
+	7750 10650 7750 11550
+Wire Wire Line
+	7750 11550 7450 11550
+$Comp
+L LED D?
+U 1 1 5A0E6C13
+P 7900 10650
+F 0 "D?" H 7900 10750 50  0001 C CNN
+F 1 "STATUS LED" H 7900 10500 50  0000 C CNN
+F 2 "" H 7900 10650 50  0001 C CNN
+F 3 "" H 7900 10650 50  0001 C CNN
+	1    7900 10650
+	-1   0    0    1
+$EndComp
+$Comp
+L GND #PWR?
+U 1 1 5A0E6C40
+P 8050 10650
+F 0 "#PWR?" H 8050 10400 50  0001 C CNN
+F 1 "GND" H 8050 10500 50  0000 C CNN
+F 2 "" H 8050 10650 50  0001 C CNN
+F 3 "" H 8050 10650 50  0001 C CNN
+	1    8050 10650
+	1    0    0    -1
+$EndComp
